Commit message: finished checkpoint

File: rhodent_description/urdf/rhodent_properties.xacro (robot description, xacro)
@@ -13,5 +13,6 @@
     <xacro:property name="LEFT_WHEEL_TRANSL" value="0 0.101 0"/>
     <xacro:property name="LEFT_WHEEL_ROT" value="-${PId2} 0 0"/>
-    <xacro:property name="CHASSIS_TO_LIDAR" value="-0.02307 0 0.1341"/>
+    <!-- <xacro:property name="CHASSIS_TO_LIDAR" value="-0.02307 0 0.1341"/> -->
+    <xacro:property name="CHASSIS_TO_LIDAR" value="0 0 0.1341"/>
     <xacro:property name="CHASSIS_TO_IMU" value="0.035 0 0.05"/>
     <!-- Joint Properties -->

File: rhodent_description/urdf/rplidar_a1.xacro (robot description, xacro)
@@ -30,5 +30,5 @@
                     <scan>
                         <horizontal>
-                            <samples>800</samples>
+                            <samples>2000</samples>
                             <resolution>1</resolution>
                             <min_angle>-3.14159265359</min_angle>
@@ -39,5 +39,5 @@
                             <min>0.10</min>
                             <max>12.0</max>
-                            <resolution>0.0174533</resolution>
+                            <resolution>0.001</resolution>
                         </range>
                     <noise>
@@ -48,5 +48,5 @@
                             reading. -->
                         <mean>0.0</mean>
-                        <stddev>0.01</stddev>
+                        <stddev>0.005</stddev>
                     </noise>
                 </ray>
