Commit message: Working teleop on gazebo

File: rhodent_description/urdf/rhodent.xacro (robot description, xacro)
@@ -1,5 +1,4 @@
 <?xml version="1.0"?>
 <robot name="Rhodent502" xmlns:xacro="http://www.ros.org/wiki/xacro">
-    <static>false</static>
     <gazebo>
         <plugin name="gazebo_ros_control" filename="libgazebo_ros_control.so">
@@ -13,11 +12,11 @@
         <color rgba="0.7 0.7 0.7 1"/>
     </material>
-    <xacro:include filename="$(find rhodent_description)/urdf/rhodent_properties.xacro" />
+    <xacro:include filename="$(find rhodent_description)/urdf/rhodent_properties.xacro"/>
     <xacro:include filename="$(find rhodent_description)/urdf/rhodent_wheel.xacro" />
-    <xacro:include filename="$(find rhodent_description)/urdf/rhodent_chassis.xacro" />
-    <!-- <link name="world"/> -->
+    <xacro:include filename="$(find rhodent_description)/urdf/rhodent_chassis.xacro"/>
+    <link name="map"/>
     <xacro:rhodent_chassis
         name = "base"
-        parent = "world"
+        parent = "map"
         color = "dark_grey"/>
     <xacro:rhodent_wheel

File: rhodent_description/urdf/rhodent_chassis.xacro (robot description, xacro)
@@ -54,9 +54,9 @@
             </collision>
         </link>
-        <!-- <joint name="${parent}_to_${name}_footprint" type="fixed">
+        <joint name="${parent}_to_${name}_footprint" type="fixed">
             <parent link="${parent}"/>
             <child link="${name}_footprint"/>
             <origin rpy="0 0 0" xyz="0 0 0"/>
-        </joint> -->
+        </joint>
         <joint name="${name}_footprint_to_${name}_link" type="fixed">
             <parent link="${name}_footprint"/>
@@ -75,6 +75,6 @@
         </joint>
         <gazebo reference="${name}_link">
-            <mu1>0.05</mu1>
-            <mu2>0.05</mu2>
+            <mu1>0.5</mu1>
+            <mu2>0.5</mu2>
             <material>Gazebo/Grey</material>
         </gazebo>
@@ -82,4 +82,6 @@
             <mu1>0</mu1>
             <mu2>0</mu2>
+            <slip1>1.0</slip1>
+            <slip2>1.0</slip2>
             <material>Gazebo/Grey</material>
         </gazebo>
@@ -87,4 +89,6 @@
             <mu1>0</mu1>
             <mu2>0</mu2>
+            <slip1>1.0</slip1>
+            <slip2>1.0</slip2>
             <material>Gazebo/Grey</material>
         </gazebo>

File: rhodent_description/urdf/rhodent_properties.xacro (robot description, xacro)
@@ -6,6 +6,8 @@
 	<!-- Geometric Properties -->
     <xacro:property name="WHEEL_RADIUS" value="0.03225"/>
+    <xacro:property name="WHEEL_SEPARATION" value="0.202"/>
 	<xacro:property name="BELLY_HEIGHT" value="0.00525"/>
-    <xacro:property name="FLOOR_TO_BASE" value="0.03225"/>
+    <!-- <xacro:property name="FLOOR_TO_BASE" value="0.03225"/> -->
+    <xacro:property name="FLOOR_TO_BASE" value="0.14225"/>
     <xacro:property name="RIGHT_WHEEL_TRANSL" value="0 -0.101 0"/>
     <xacro:property name="RIGHT_WHEEL_ROT" value="-${PId2} 0 0"/>
@@ -15,7 +17,7 @@
     <xacro:property name="U_MAX" value="3.0"/>
     <xacro:property name="V_MAX" value="12.0"/>
-    <xacro:property name="WHEEL_JOINT_DAMP" value="0.02"/>
+    <xacro:property name="WHEEL_JOINT_DAMP" value="0.3"/>
     <!-- Inertial Properties -->
-    <xacro:property name="CHASSIS_COM" value="-0.02718 -0.00201 -0.02"/>
+    <xacro:property name="CHASSIS_COM" value="-0.02718 -0.00201 -0.002"/>
     <xacro:property name="CHASSIS_Ixx" value="0.009607873"/>
     <xacro:property name="CHASSIS_Iyy" value="0.010242986"/>
@@ -26,10 +28,10 @@
     <xacro:property name="CHASSIS_M" value="1.6015"/>
     <xacro:property name="WHEEL_COM" value="0 0 -0.00039"/>
-    <xacro:property name="WHEEL_Ixx" value="0.000032052"/>
-    <xacro:property name="WHEEL_Iyy" value="0.000032052"/>
-    <xacro:property name="WHEEL_Izz" value="0.000059397"/>
-    <xacro:property name="WHEEL_Ixy" value="0.000000001"/>
-    <xacro:property name="WHEEL_Iyz" value="0.000000001"/>
-    <xacro:property name="WHEEL_Ixz" value="0.000000001"/>
+    <xacro:property name="WHEEL_Ixx" value="0.00012052"/>
+    <xacro:property name="WHEEL_Iyy" value="0.00012052"/>
+    <xacro:property name="WHEEL_Izz" value="0.0029397"/>
+    <xacro:property name="WHEEL_Ixy" value="0.0"/>
+    <xacro:property name="WHEEL_Iyz" value="0.0"/>
+    <xacro:property name="WHEEL_Ixz" value="0.0"/>
     <xacro:property name="WHEEL_M" value="0.11"/>
 </robot>

File: rhodent_description/urdf/rhodent_wheel.xacro (robot description, xacro)
@@ -5,7 +5,7 @@
         <link name="${name}">
             <inertial>
-                <origin rpy="0 0 0" xyz="0 0 0"/>
-                <mass value="0.11" />
-                <inertia ixx="0.000032052" ixy="0.000032052" ixz="0.000032052" iyy="0.000032052" iyz="0.0000032052" izz="0.000059397"/>
+                <origin rpy="0 0 0" xyz="${WHEEL_COM}"/>
+                <mass value="${WHEEL_M}" />
+                <inertia ixx="${WHEEL_Ixx}" ixy="${WHEEL_Ixy}" ixz="${WHEEL_Ixz}" iyy="${WHEEL_Iyy}" iyz="${WHEEL_Iyz}" izz="${WHEEL_Izz}"/>
             </inertial>
             <visual>
@@ -32,6 +32,8 @@
         </joint>
         <gazebo reference="${name}">
-            <mu1>0.001</mu1>
-            <mu2>0.001</mu2>
+            <mu1>0.7</mu1>
+            <mu2>0.7</mu2>
+            <slip1>0.2</slip1>
+            <slip2>0.2</slip2>
             <material>Gazebo/Grey</material>
         </gazebo>

Commit message: diff_kinematics node done

File: rhodent_description/urdf/rhodent.xacro (robot description, xacro)
@@ -15,8 +15,8 @@
     <xacro:include filename="$(find rhodent_description)/urdf/rhodent_wheel.xacro" />
     <xacro:include filename="$(find rhodent_description)/urdf/rhodent_chassis.xacro"/>
-    <link name="map"/>
+    <link name="odom"/>
     <xacro:rhodent_chassis
         name = "base"
-        parent = "map"
+        parent = "odom"
         color = "dark_grey"/>
     <xacro:rhodent_wheel

File: rhodent_description/urdf/rhodent_chassis.xacro (robot description, xacro)
@@ -18,7 +18,7 @@
             </visual>
             <collision name="collision">
-                <origin rpy="0 0 0" xyz="-0.02 0 0.12"/>
+                <origin rpy="0 0 0" xyz="-0.03 0 0.12"/>
                 <geometry>
-                    <cylinder radius = "0.089" length = "0.290"/>
+                    <cylinder radius = "0.1" length = "0.290"/>
                 </geometry>
             </collision>

File: rhodent_description/urdf/rhodent_properties.xacro (robot description, xacro)
@@ -8,6 +8,5 @@
     <xacro:property name="WHEEL_SEPARATION" value="0.202"/>
 	<xacro:property name="BELLY_HEIGHT" value="0.00525"/>
-    <!-- <xacro:property name="FLOOR_TO_BASE" value="0.03225"/> -->
-    <xacro:property name="FLOOR_TO_BASE" value="0.14225"/>
+    <xacro:property name="FLOOR_TO_BASE" value="0.03225"/>
     <xacro:property name="RIGHT_WHEEL_TRANSL" value="0 -0.101 0"/>
     <xacro:property name="RIGHT_WHEEL_ROT" value="-${PId2} 0 0"/>
@@ -15,6 +14,6 @@
     <xacro:property name="LEFT_WHEEL_ROT" value="-${PId2} 0 0"/>
     <!-- Joint Properties -->
-    <xacro:property name="U_MAX" value="3.0"/>
-    <xacro:property name="V_MAX" value="12.0"/>
+    <xacro:property name="U_MAX" value="10.0"/>
+    <xacro:property name="V_MAX" value="20.0"/>
     <xacro:property name="WHEEL_JOINT_DAMP" value="0.3"/>
     <!-- Inertial Properties -->

Commit message: add rplidar a1

File: rhodent_description/urdf/rhodent.xacro (robot description, xacro)
@@ -15,4 +15,5 @@
     <xacro:include filename="$(find rhodent_description)/urdf/rhodent_wheel.xacro" />
     <xacro:include filename="$(find rhodent_description)/urdf/rhodent_chassis.xacro"/>
+    <xacro:include filename="$(find rhodent_description)/urdf/rplidar_a1.xacro"/>
     <link name="odom"/>
     <xacro:rhodent_chassis
@@ -34,3 +35,9 @@
         color = "aluminium"
         rotate = "${PI}"/>
+    <xacro:rplidar_a1
+        prefix = "top"
+        parent = "base_link"
+        offset_from_parent = "${CHASSIS_TO_LIDAR}"
+        visualize = "true"
+        color = "dark_grey"/>
 </robot>

File: rhodent_description/urdf/rhodent_chassis.xacro (robot description, xacro)
@@ -18,7 +18,7 @@
             </visual>
             <collision name="collision">
-                <origin rpy="0 0 0" xyz="-0.03 0 0.12"/>
+                <origin rpy="0 0 0" xyz="-0.03 0 0.03"/>
                 <geometry>
-                    <cylinder radius = "0.1" length = "0.290"/>
+                    <cylinder radius = "0.1" length = "0.11"/>
                 </geometry>
             </collision>

File: rhodent_description/urdf/rhodent_properties.xacro (robot description, xacro)
@@ -13,4 +13,5 @@
     <xacro:property name="LEFT_WHEEL_TRANSL" value="0 0.101 0"/>
     <xacro:property name="LEFT_WHEEL_ROT" value="-${PId2} 0 0"/>
+    <xacro:property name="CHASSIS_TO_LIDAR" value="-0.02307 0 0.1341"/>
     <!-- Joint Properties -->
     <xacro:property name="U_MAX" value="10.0"/>

File: rhodent_description/urdf/rhodent_wheel.xacro (robot description, xacro)
@@ -32,6 +32,6 @@
         </joint>
         <gazebo reference="${name}">
-            <mu1>0.7</mu1>
-            <mu2>0.7</mu2>
+            <mu1>0.8</mu1>
+            <mu2>0.8</mu2>
             <slip1>0.2</slip1>
             <slip2>0.2</slip2>

Commit message: add move_base

File: rhodent_description/urdf/rhodent.xacro (robot description, xacro)
@@ -16,5 +16,11 @@
     <xacro:include filename="$(find rhodent_description)/urdf/rhodent_chassis.xacro"/>
     <xacro:include filename="$(find rhodent_description)/urdf/rplidar_a1.xacro"/>
-    <link name="odom"/>
+    <xacro:include filename="$(find rhodent_description)/urdf/6dof_imu.xacro"/>
+    <!-- <link name="map"/>
+    <joint name="map_to_odom" type="fixed">
+        <parent link="map"/>
+        <child link="odom"/>
+    </joint>
+    <link name="odom"/> -->
     <xacro:rhodent_chassis
         name = "base"
@@ -39,5 +45,12 @@
         parent = "base_link"
         offset_from_parent = "${CHASSIS_TO_LIDAR}"
+        visualize = "false"
+        color = "dark_grey"
+        topic = "/rhodent/scan"/>
+    <xacro:imu
+        prefix = "main"
+        parent = "base_link"
+        offset_from_parent = "${CHASSIS_TO_IMU}"
         visualize = "true"
-        color = "dark_grey"/>
+        topic = "/rhodent/imu"/>
 </robot>

File: rhodent_description/urdf/rhodent_chassis.xacro (robot description, xacro)
@@ -54,9 +54,10 @@
             </collision>
         </link>
+<!--
         <joint name="${parent}_to_${name}_footprint" type="fixed">
             <parent link="${parent}"/>
             <child link="${name}_footprint"/>
             <origin rpy="0 0 0" xyz="0 0 0"/>
-        </joint>
+        </joint> -->
         <joint name="${name}_footprint_to_${name}_link" type="fixed">
             <parent link="${name}_footprint"/>
@@ -72,5 +73,5 @@
             <parent link="${name}_link"/>
             <child link="${name}_fcaster"/>
-            <origin rpy="0 0 0" xyz="0.03723 0 -0.0243"/>
+            <origin rpy="0 0 0" xyz="0.03723 0 -0.0255"/>
         </joint>
         <gazebo reference="${name}_link">

File: rhodent_description/urdf/rhodent_properties.xacro (robot description, xacro)
@@ -14,4 +14,5 @@
     <xacro:property name="LEFT_WHEEL_ROT" value="-${PId2} 0 0"/>
     <xacro:property name="CHASSIS_TO_LIDAR" value="-0.02307 0 0.1341"/>
+    <xacro:property name="CHASSIS_TO_IMU" value="0.035 0 0.05"/>
     <!-- Joint Properties -->
     <xacro:property name="U_MAX" value="10.0"/>

File: rhodent_description/urdf/rplidar_a1.xacro (robot description, xacro)
@@ -2,5 +2,5 @@
 <robot name="rplidar_a1" xmlns:xacro="http://www.ros.org/wiki/xacro">
     <xacro:include filename="$(find rhodent_description)/urdf/rhodent_properties.xacro" />
-    <xacro:macro name="rplidar_a1" params="prefix parent offset_from_parent visualize color">
+    <xacro:macro name="rplidar_a1" params="prefix parent offset_from_parent visualize color topic">
         <joint name="${prefix}_rplidar_joint" type="fixed">
             <origin xyz="${offset_from_parent}" rpy="0 0 0"/>
@@ -52,5 +52,5 @@
                 </ray>
                 <plugin name="gazebo_ros_${prefix}_lidar" filename="libgazebo_ros_laser.so">
-                    <topicName>/rhodent/${prefix}_laser/scan</topicName>
+                    <topicName>${topic}</topicName>
                     <frameName>${prefix}_rplidar_link</frameName>
                 </plugin>

Commit message: fine tuning the local planner

File: rhodent_description/urdf/rhodent.xacro (robot description, xacro)
@@ -17,13 +17,7 @@
     <xacro:include filename="$(find rhodent_description)/urdf/rplidar_a1.xacro"/>
     <xacro:include filename="$(find rhodent_description)/urdf/6dof_imu.xacro"/>
-    <!-- <link name="map"/>
-    <joint name="map_to_odom" type="fixed">
-        <parent link="map"/>
-        <child link="odom"/>
-    </joint>
-    <link name="odom"/> -->
     <xacro:rhodent_chassis
         name = "base"
-        parent = "odom"
+        parent = "None"
         color = "dark_grey"/>
     <xacro:rhodent_wheel

File: rhodent_description/urdf/rhodent_properties.xacro (robot description, xacro)
@@ -15,9 +15,9 @@
     <!-- <xacro:property name="CHASSIS_TO_LIDAR" value="-0.02307 0 0.1341"/> -->
     <xacro:property name="CHASSIS_TO_LIDAR" value="0 0 0.1341"/>
-    <xacro:property name="CHASSIS_TO_IMU" value="0.035 0 0.05"/>
+    <xacro:property name="CHASSIS_TO_IMU" value="0 0 0.05"/>
     <!-- Joint Properties -->
     <xacro:property name="U_MAX" value="10.0"/>
     <xacro:property name="V_MAX" value="20.0"/>
-    <xacro:property name="WHEEL_JOINT_DAMP" value="0.3"/>
+    <xacro:property name="WHEEL_JOINT_DAMP" value="0.2"/>
     <!-- Inertial Properties -->
     <xacro:property name="CHASSIS_COM" value="-0.02718 -0.00201 -0.002"/>
